File: iso124-1/ios124/ios124.kicad_pcb (KiCad board)
At the start: 2 copper layers, 68.6 x 35.6 mm, 7 parts, among them J1 Screw_Terminal_01x02, J2 Screw_Terminal_01x03, J3 Screw_Terminal_01x03, J4 Screw_Terminal_01x02, U1 LM741, U2 ISO124, U3 LM741

Commit message: iso124pcb-1
Parts:
- added J1: Screw_Terminal_01x02, TerminalBlock:TerminalBlock_Altech_AK300-2_P5.00mm, F.Cu at (177.4, 137.8)
- added J1: Screw_Terminal_01x02, TerminalBlock:TerminalBlock_Altech_AK300-2_P5.00mm, F.Cu at (87.6, 139.2)
- added J1: Screw_Terminal_01x02, TerminalBlock:TerminalBlock_Altech_AK300-2_P5.00mm, F.Cu at (175.5, 81.7)
- added J2: Screw_Terminal_01x03, TerminalBlock:TerminalBlock_Altech_AK300-3_P5.00mm, F.Cu at (177.4, 123.9)
- added J2: Screw_Terminal_01x03, TerminalBlock:TerminalBlock_Altech_AK300-3_P5.00mm, F.Cu at (87.6, 125.3)
- added J2: Screw_Terminal_01x03, TerminalBlock:TerminalBlock_Altech_AK300-3_P5.00mm, F.Cu at (175.5, 67.8)
- added J3: Screw_Terminal_01x03, TerminalBlock:TerminalBlock_Altech_AK300-3_P5.00mm, F.Cu at (224.4, 113.8)
- added J3: Screw_Terminal_01x03, TerminalBlock:TerminalBlock_Altech_AK300-3_P5.00mm, F.Cu at (134.6, 115.2)
- added J3: Screw_Terminal_01x03, TerminalBlock:TerminalBlock_Altech_AK300-3_P5.00mm, F.Cu at (222.5, 57.6)
- added J4: Screw_Terminal_01x02, TerminalBlock:TerminalBlock_Altech_AK300-2_P5.00mm, F.Cu at (224.4, 132.3)
- added J4: Screw_Terminal_01x02, TerminalBlock:TerminalBlock_Altech_AK300-2_P5.00mm, F.Cu at (134.6, 133.7)
- added J4: Screw_Terminal_01x02, TerminalBlock:TerminalBlock_Altech_AK300-2_P5.00mm, F.Cu at (222.5, 76.1)
- added U1: LM741, Package_DIP:DIP-8_W7.62mm_LongPads, F.Cu at (190.1, 131.5)
- added U1: LM741, Package_DIP:DIP-8_W7.62mm_LongPads, F.Cu at (100.3, 132.9)
- added U1: LM741, Package_DIP:DIP-8_W7.62mm_LongPads, F.Cu at (188.2, 75.4)
- added U2: ISO124, Package_DIP:DIP-16_W7.62mm_LongPads, F.Cu at (191.4, 120.1)
- added U2: ISO124, Package_DIP:DIP-16_W7.62mm_LongPads, F.Cu at (101.6, 121.5)
- added U2: ISO124, Package_DIP:DIP-16_W7.62mm_LongPads, F.Cu at (189.5, 64.0)
- added U3: LM741, Package_DIP:DIP-8_W7.62mm_LongPads, F.Cu at (204.1, 131.5)
- added U3: LM741, Package_DIP:DIP-8_W7.62mm_LongPads, F.Cu at (114.3, 132.9)
- added U3: LM741, Package_DIP:DIP-8_W7.62mm_LongPads, F.Cu at (202.2, 75.4)
- moved J3 21.2 mm to (135.2, 57.4)
- moved J4 21.2 mm to (135.2, 75.9)
- moved U1 21.2 mm to (101.0, 75.1)
- moved U3 21.2 mm to (114.9, 75.1)
- moved J1 21.2 mm to (88.3, 81.4)
- moved J2 21.2 mm to (88.3, 67.5)
- moved U2 21.2 mm to (102.2, 63.7)
Routing:
- net (no net): track 0.00 -> 1206.0 mm, vias 0 -> 16
Other:
- board size 68.6 x 35.6 mm -> 158.4 x 93.4 mm
