File: igtvgtfinal/igtvgtequment/igtvgtequment.sch (KiCad schematic (older format))
At the start: 7 parts

Commit message: i
Parts:
- gave numbers to parts that had none: 7
Changed lines of the file:
@@
 EESchema Schematic File Version 4
-LIBS:IgtVgtTestEqument-cache
-LIBS:igtvgtequment-cache
 EELAYER 26 0
 EELAYER END
 $Descr A4 11693 8268
 encoding utf-8
-Sheet 3 3
+Sheet 1 1
 Title ""
 Date ""
@@
 $EndDescr
 $Comp
-L Amplifier_Operational:LM741 U?
+L Amplifier_Operational:LM741 U1
 U 1 1 5BB01E85
 P 4450 4400
-F 0 "U?" H 4791 4446 50  0000 L CNN
+F 0 "U1" H 4791 4446 50  0000 L CNN
 F 1 "LM741" H 4791 4355 50  0000 L CNN
 F 2 "" H 4500 4450 50  0001 C CNN
@@
 	3700 4500 4150 4500
 $Comp
-L Transistor_BJT:2N2219 Q?
+L Transistor_BJT:2N2219 Q1
 U 1 1 5BB02001
 P 5650 4400
-F 0 "Q?" H 5841 4446 50  0000 L CNN
+F 0 "Q1" H 5841 4446 50  0000 L CNN
 F 1 "2N2219" H 5841 4355 50  0000 L CNN
 F 2 "Package_TO_SOT_THT:TO-39-3" H 5850 4325 50  0001 L CIN
@@
 GND
 $Comp
-L Device:R R?
+L Device:R R1
 U 1 1 5BB020F4
 P 5100 4400
-F 0 "R?" V 4893 4400 50  0000 C CNN
+F 0 "R1" V 4893 4400 50  0000 C CNN
 F 1 "R" V 4984 4400 50  0000 C CNN
 F 2 "" V 5030 4400 50  0001 C CNN
@@
 	4950 4400 4750 4400
 $Comp
-L Device:R R?
+L Device:R R2
 U 1 1 5BB022CA
 P 5750 3400
-F 0 "R?" H 5680 3354 50  0000 R CNN
+F 0 "R2" H 5680 3354 50  0000 R CNN
 F 1 "R" H 5680 3445 50  0000 R CNN
 F 2 "" V 5680 3400 50  0001 C CNN
@@
 	5750 3650 5750 4000
 $Comp
-L Amplifier_Operational:LM741 U?
+L Amplifier_Operational:LM741 U2
 U 1 1 5BB027C7
 P 6800 3900
-F 0 "U?" H 7141 3946 50  0000 L CNN
+F 0 "U2" H 7141 3946 50  0000 L CNN
 F 1 "LM741" H 7141 3855 50  0000 L CNN
 F 2 "" H 6850 3950 50  0001 C CNN
@@
 	5750 4000 5750 4200
 $Comp
-L Transistor_FET:IRF9540N Q?
+L Transistor_FET:IRF9540N Q2
 U 1 1 5BB0298A
 P 7650 3900
-F 0 "Q?" H 7855 3854 50  0000 L CNN
+F 0 "Q2" H 7855 3854 50  0000 L CNN
 F 1 "IRF9540N" H 7855 3945 50  0000 L CNN
 F 2 "Package_TO_SOT_THT:TO-220-3_Vertical" H 7850 3825 50  0001 L CIN
@@
 -15VDC
 $Comp
-L Device:R R?
+L Device:R R3
 U 1 1 5BB02D52
 P 7750 3050
-F 0 "R?" H 7680 3004 50  0000 R CNN
+F 0 "R3" H 7680 3004 50  0000 R CNN
 F 1 "R" H 7680 3095 50  0000 R CNN
 F 2 "" V 7680 3050 50  0001 C CNN
