File: 门极测试台/IgtVgtTestEqument/IgtVgtTestEqument.sch (KiCad schematic (older format))
At the start: 2 parts, among them J1 Screw_Terminal_01x03, SW1 SW_Push

Commit message: i
Changed lines of the file:
@@
 EESchema Schematic File Version 4
 LIBS:IgtVgtTestEqument-cache
+LIBS:igtvgtequment-cache
 EELAYER 26 0
 EELAYER END
@@
 F8 "K" O R 5750 3100 50
 F9 "DC5V" I L 4550 2850 50
+F10 "+15VDC" I L 4550 2450 50
 $EndSheet
 Wire Wire Line
