File: 单片机/单片机门极/单片机门极.sch (KiCad schematic (older format))
At the start: 9 parts, among them J1 Screw_Terminal_01x02, U1 L7805

Commit message: 741
Parts:
- removed U?: stc15w408as, Package_DIP:DIP-20_W7.62mm_LongPads, symbol kicadsch:stc15w408as
- added C5: C, symbol Device:C
- added D2, D3, D4, D5: 1N4007, Diode_THT:D_DO-41_SOD81_P10.16mm_Horizontal, symbol Diode:1N4007
- added J2, J3: Screw_Terminal_01x02, symbol Connector:Screw_Terminal_01x02
- added Q1: IRF540N, Package_TO_SOT_THT:TO-220-3_Vertical, symbol Transistor_FET:IRF540N
- added Q2: BF244A, Package_TO_SOT_THT:TO-92_Inline, symbol Transistor_FET:BF244A
- added Q3: IRF9540N, Package_TO_SOT_THT:TO-220-3_Vertical, symbol Transistor_FET:IRF9540N
- added R10, R11, R12, R13, R14, R2, R3, R4, R5, R6, R7, R8, R9: R, symbol Device:R
- added U2: stc15w408as, Package_DIP:DIP-20_W7.62mm_LongPads, symbol kicadsch:stc15w408as
- added U3: MCP4822, symbol Analog_DAC:MCP4822
- added U4, U5, U6: LM741, symbol Amplifier_Operational:LM741
Connections:
- net labels added: +15V, -15V
- wire segments 25 -> 105
- no-connect marks 0 -> 1
Other:
- note added: "DAC"
- note added: "MCU"

Commit message: igtvgtpower
Parts:
- removed J2, J3: Screw_Terminal_01x02, symbol Connector:Screw_Terminal_01x02
- added D6, D7: 1N4148, Diode_THT:D_DO-35_SOD27_P7.62mm_Horizontal, symbol Diode:1N4148
- added J?: Screw_Terminal_01x04, symbol Connector:Screw_Terminal_01x04
- added K1, K2: RELAY-5, Relay_THT:Relay_DPDT_FRT5, symbol kicadsch:RELAY-5
- added Q4, Q5: IRF540N, Package_TO_SOT_THT:TO-220-3_Vertical, symbol Transistor_FET:IRF540N
- added Q6: TIC126, Package_TO_SOT_THT:TO-220-3_Vertical, symbol Triac_Thyristor:TIC126
- added R15, R16, R17: R, symbol Device:R
- added SW?: SW_Push, symbol Switch:SW_Push
Connections:
- net labels added: +12V
- wire segments 105 -> 145
Other:
- note added: "A"
- note added: "DUT"
- note added: "G"
- note added: "IGT OUTPUT"
- note added: "K"
- note added: "Program"
- note added: "VGT OUTPUT"
- note added: "anode select"
- note added: "igt unit"
- note added: "igt/vgt select"
- note added: "vgt unit"
- moved on the sheet: Q1, U3

Commit message: display
Parts:
- added C10, C11, C14, C16, C6, C7: CP1, symbol Device:CP1
- added C12, C13, C15, C17, C8, C9: C, symbol Device:C
- added D10, D11, D14, D15, D16, D17, D8, D9: 1N4007, Diode_THT:D_DO-41_SOD81_P10.16mm_Horizontal, symbol Diode:1N4007
- added D12, D13, D18: LED, symbol Device:LED
- added DS1: 128*64, LCD128*64, symbol kicadsch:128*64
- added J3: Screw_Terminal_01x03, symbol Connector:Screw_Terminal_01x03
- added J4: Screw_Terminal_01x02, kipcblib:CON2liubiao, symbol Connector:Screw_Terminal_01x02
- added R18, R19, R20, R21, R22, R23: R, symbol Device:R
- added U10: L7812, symbol Regulator_Linear:L7812
- added U7: LM7815_TO220, Package_TO_SOT_THT:TO-220-3_Vertical, symbol Regulator_Linear:LM7815_TO220
- added U8: L7915, symbol Regulator_Linear:L7915
- added U9: LM311, symbol Comparator:LM311
- gave numbers to parts that had none: 2
Connections:
- net labels added: pass_fail_select
- wire segments 145 -> 258
Other:
- moved on the sheet: D2, D3, D4, D5, Q1, Q4, Q5, Q6, U3

Commit message: foot
Parts:
- removed R18, R19, R23: R, symbol Device:R
- added R? (x3): R, Resistor_THT:R_Axial_DIN0309_L9.0mm_D3.2mm_P20.32mm_Horizontal, symbol Device:R
- R1: footprint (none) -> Resistor_THT:R_Axial_DIN0309_L9.0mm_D3.2mm_P20.32mm_Horizontal
- R6: value R -> (none)
Changed lines of the file:
@@
 F 0 "R1" H 6070 2196 50  0000 L CNN
 F 1 "R" H 6070 2105 50  0000 L CNN
-F 2 "" V 5930 2150 50  0001 C CNN
+F 2 "Resistor_THT:R_Axial_DIN0309_L9.0mm_D3.2mm_P20.32mm_Horizontal" V 5930 2150 50  0001 C CNN
 F 3 "~" H 6000 2150 50  0001 C CNN
 	1    6000 2150
@@
 P 8750 7800
 F 0 "R6" V 8543 7800 50  0000 C CNN
-F 1 "R" V 8634 7800 50  0000 C CNN
+F 1 "" V 8634 7800 50  0000 C CNN
 F 2 "" V 8680 7800 50  0001 C CNN
 F 3 "~" H 8750 7800 50  0001 C CNN
@@
 GND
 $Comp
-L Device:R R18
-U 1 1 5BCB1AC0
-P 12000 1600
-F 0 "R18" H 12070 1646 50  0000 L CNN
-F 1 "R" H 12070 1555 50  0000 L CNN
-F 2 "" V 11930 1600 50  0001 C CNN
-F 3 "~" H 12000 1600 50  0001 C CNN
-	1    12000 1600
-	1    0    0    -1
-$EndComp
-$Comp
 L Device:LED D12
 U 1 1 5BCB1AC7
@@
 Connection ~ 11100 3350
 $Comp
-L Device:R R19
-U 1 1 5BD598BA
-P 12000 2600
-F 0 "R19" H 12070 2646 50  0000 L CNN
-F 1 "R" H 12070 2555 50  0000 L CNN
-F 2 "" V 11930 2600 50  0001 C CNN
-F 3 "~" H 12000 2600 50  0001 C CNN
-	1    12000 2600
-	1    0    0    -1
-$EndComp
-$Comp
 L Device:LED D13
 U 1 1 5BD598C1
@@
 GND
 $Comp
-L Device:R R23
-U 1 1 5BD848A7
-P 18900 2150
-F 0 "R23" H 18970 2196 50  0000 L CNN
-F 1 "R" H 18970 2105 50  0000 L CNN
-F 2 "" V 18830 2150 50  0001 C CNN
-F 3 "~" H 18900 2150 50  0001 C CNN
-	1    18900 2150
-	1    0    0    -1
-$EndComp
-$Comp
 L Device:LED D18
 U 1 1 5BD848AE
@@
 Text Notes 7250 2700 0    50   ~ 0
 INPUT-AC
+$Comp
+L Device:R R?
+U 1 1 5BC719BD
+P 12000 1600
+F 0 "R?" H 12070 1646 50  0000 L CNN
+F 1 "R" H 12070 1555 50  0000 L CNN
+F 2 "Resistor_THT:R_Axial_DIN0309_L9.0mm_D3.2mm_P20.32mm_Horizontal" V 11930 1600 50  0001 C CNN
+F 3 "~" H 12000 1600 50  0001 C CNN
+	1    12000 1600
+	1    0    0    -1
+$EndComp
+$Comp
+L Device:R R?
+U 1 1 5BC71C3B
+P 12000 2600
+F 0 "R?" H 12070 2646 50  0000 L CNN
+F 1 "R" H 12070 2555 50  0000 L CNN
+F 2 "Resistor_THT:R_Axial_DIN0309_L9.0mm_D3.2mm_P20.32mm_Horizontal" V 11930 2600 50  0001 C CNN
+F 3 "~" H 12000 2600 50  0001 C CNN
+	1    12000 2600
+	1    0    0    -1
+$EndComp
+$Comp
+L Device:R R?
+U 1 1 5BC729E1
+P 18900 2150
+F 0 "R?" H 18970 2196 50  0000 L CNN
+F 1 "R" H 18970 2105 50  0000 L CNN
+F 2 "Resistor_THT:R_Axial_DIN0309_L9.0mm_D3.2mm_P20.32mm_Horizontal" V 18830 2150 50  0001 C CNN
+F 3 "~" H 18900 2150 50  0001 C CNN
+	1    18900 2150
+	1    0    0    -1
+$EndComp
 $EndSCHEMATC

Commit message: rfootpage
Parts:
- R10, R11, R12, R13, R14, R15, R16, R17, R2, R20, R21, R22, R3, R4, R5, R7, R8, R9: footprint (none) -> Resistor_THT:R_Axial_DIN0309_L9.0mm_D3.2mm_P20.32mm_Horizontal
- R6: value (none) -> ~; footprint (none) -> Resistor_THT:R_Axial_DIN0309_L9.0mm_D3.2mm_P20.32mm_Horizontal
- gave numbers to parts that had none: 3
Changed lines of the file:
@@
 -15V
 Wire Wire Line
-	8950 7150 9300 7150
-Wire Wire Line
 	8350 7250 8150 7250
-Wire Wire Line
-	9300 7800 9300 7150
-Connection ~ 9300 7150
 $Comp
 L Device:R R2
@@
 F 0 "R2" V 7843 7050 50  0000 C CNN
 F 1 "R" V 7934 7050 50  0000 C CNN
-F 2 "" V 7980 7050 50  0001 C CNN
+F 2 "Resistor_THT:R_Axial_DIN0309_L9.0mm_D3.2mm_P20.32mm_Horizontal" V 7980 7050 50  0001 C CNN
 F 3 "~" H 8050 7050 50  0001 C CNN
 	1    8050 7050
@@
 P 8750 7800
 F 0 "R6" V 8543 7800 50  0000 C CNN
-F 1 "" V 8634 7800 50  0000 C CNN
-F 2 "" V 8680 7800 50  0001 C CNN
+F 1 "~" V 8634 7800 50  0000 C CNN
+F 2 "Resistor_THT:R_Axial_DIN0309_L9.0mm_D3.2mm_P20.32mm_Horizontal" V 8680 7800 50  0001 C CNN
 F 3 "~" H 8750 7800 50  0001 C CNN
 	1    8750 7800
@@
 F 0 "R4" H 8220 8046 50  0000 L CNN
 F 1 "R" H 8220 7955 50  0000 L CNN
-F 2 "" V 8080 8000 50  0001 C CNN
+F 2 "Resistor_THT:R_Axial_DIN0309_L9.0mm_D3.2mm_P20.32mm_Horizontal" V 8080 8000 50  0001 C CNN
 F 3 "~" H 8150 8000 50  0001 C CNN
 	1    8150 8000
@@
 Wire Wire Line
 	8200 7050 8350 7050
-Wire Wire Line
-	8900 7800 9300 7800
 Wire Wire Line
 	8600 7800 8150 7800
@@
 F 0 "R3" V 7893 9250 50  0000 C CNN
 F 1 "R" V 7984 9250 50  0000 C CNN
-F 2 "" V 8030 9250 50  0001 C CNN
+F 2 "Resistor_THT:R_Axial_DIN0309_L9.0mm_D3.2mm_P20.32mm_Horizontal" V 8030 9250 50  0001 C CNN
 F 3 "~" H 8100 9250 50  0001 C CNN
 	1    8100 9250
@@
 F 0 "R7" V 8593 10000 50  0000 C CNN
 F 1 "R" V 8684 10000 50  0000 C CNN
-F 2 "" V 8730 10000 50  0001 C CNN
+F 2 "Resistor_THT:R_Axial_DIN0309_L9.0mm_D3.2mm_P20.32mm_Horizontal" V 8730 10000 50  0001 C CNN
 F 3 "~" H 8800 10000 50  0001 C CNN
 	1    8800 10000
@@
 F 0 "R5" H 8270 10246 50  0000 L CNN
 F 1 "R" H 8270 10155 50  0000 L CNN
-F 2 "" V 8130 10200 50  0001 C CNN
+F 2 "Resistor_THT:R_Axial_DIN0309_L9.0mm_D3.2mm_P20.32mm_Horizontal" V 8130 10200 50  0001 C CNN
 F 3 "~" H 8200 10200 50  0001 C CNN
 	1    8200 10200
@@
 F 0 "R8" V 9493 7150 50  0000 C CNN
 F 1 "R" V 9584 7150 50  0000 C CNN
-F 2 "" V 9630 7150 50  0001 C CNN
+F 2 "Resistor_THT:R_Axial_DIN0309_L9.0mm_D3.2mm_P20.32mm_Horizontal" V 9630 7150 50  0001 C CNN
 F 3 "~" H 9700 7150 50  0001 C CNN
 	1    9700 7150
 	0    1    1    0
 $EndComp
-Wire Wire Line
-	9300 7150 9550 7150
 Wire Wire Line
 	9850 7150 9950 7150
@@
 F 0 "R10" H 10320 6696 50  0000 L CNN
 F 1 "R" H 10320 6605 50  0000 L CNN
-F 2 "" V 10180 6650 50  0001 C CNN
+F 2 "Resistor_THT:R_Axial_DIN0309_L9.0mm_D3.2mm_P20.32mm_Horizontal" V 10180 6650 50  0001 C CNN
 F 3 "~" H 10250 6650 50  0001 C CNN
 	1    10250 6650
@@
 F 0 "R11" H 10320 7696 50  0000 L CNN
 F 1 "R" H 10320 7605 50  0000 L CNN
-F 2 "" V 10180 7650 50  0001 C CNN
+F 2 "Resistor_THT:R_Axial_DIN0309_L9.0mm_D3.2mm_P20.32mm_Horizontal" V 10180 7650 50  0001 C CNN
 F 3 "~" H 10250 7650 50  0001 C CNN
 	1    10250 7650
@@
 F 0 "R9" V 9493 9350 50  0000 C CNN
 F 1 "R" V 9584 9350 50  0000 C CNN
-F 2 "" V 9630 9350 50  0001 C CNN
+F 2 "Resistor_THT:R_Axial_DIN0309_L9.0mm_D3.2mm_P20.32mm_Horizontal" V 9630 9350 50  0001 C CNN
 F 3 "~" H 9700 9350 50  0001 C CNN
 	1    9700 9350
@@
 F 0 "R12" H 10280 8754 50  0000 R CNN
 F 1 "R" H 10280 8845 50  0000 R CNN
-F 2 "" V 10280 8800 50  0001 C CNN
+F 2 "Resistor_THT:R_Axial_DIN0309_L9.0mm_D3.2mm_P20.32mm_Horizontal" V 10280 8800 50  0001 C CNN
 F 3 "~" H 10350 8800 50  0001 C CNN
 	1    10350 8800
@@
 F 0 "R13" H 10280 10004 50  0000 R CNN
 F 1 "R" H 10280 10095 50  0000 R CNN
-F 2 "" V 10280 10050 50  0001 C CNN
+F 2 "Resistor_THT:R_Axial_DIN0309_L9.0mm_D3.2mm_P20.32mm_Horizontal" V 10280 10050 50  0001 C CNN
 F 3 "~" H 10350 10050 50  0001 C CNN
 	1    10350 10050
@@
 F 0 "R14" H 12480 8404 50  0000 R CNN
 F 1 "R" H 12480 8495 50  0000 R CNN
-F 2 "" V 12480 8450 50  0001 C CNN
+F 2 "Resistor_THT:R_Axial_DIN0309_L9.0mm_D3.2mm_P20.32mm_Horizontal" V 12480 8450 50  0001 C CNN
 F 3 "~" H 12550 8450 50  0001 C CNN
 	1    12550 8450
@@
 F 0 "R15" H 14820 6896 50  0000 L CNN
 F 1 "R" H 14820 6805 50  0000 L CNN
-F 2 "" V 14680 6850 50  0001 C CNN
+F 2 "Resistor_THT:R_Axial_DIN0309_L9.0mm_D3.2mm_P20.32mm_Horizontal" V 14680 6850 50  0001 C CNN
 F 3 "~" H 14750 6850 50  0001 C CNN
 	1    14750 6850
@@
 F 0 "R16" V 5143 11400 50  0000 C CNN
 F 1 "R" V 5234 11400 50  0000 C CNN
-F 2 "" V 5280 11400 50  0001 C CNN
+F 2 "Resistor_THT:R_Axial_DIN0309_L9.0mm_D3.2mm_P20.32mm_Horizontal" V 5280 11400 50  0001 C CNN
 F 3 "~" H 5350 11400 50  0001 C CNN
 	1    5350 11400
@@
 F 0 "R17" V 6143 11400 50  0000 C CNN
 F 1 "R" V 6234 11400 50  0000 C CNN
-F 2 "" V 6280 11400 50  0001 C CNN
+F 2 "Resistor_THT:R_Axial_DIN0309_L9.0mm_D3.2mm_P20.32mm_Horizontal" V 6280 11400 50  0001 C CNN
 F 3 "~" H 6350 11400 50  0001 C CNN
 	1    6350 11400
@@
 F 0 "R20" H 15870 9196 50  0000 L CNN
 F 1 "R" H 15870 9105 50  0000 L CNN
-F 2 "" V 15730 9150 50  0001 C CNN
+F 2 "Resistor_THT:R_Axial_DIN0309_L9.0mm_D3.2mm_P20.32mm_Horizontal" V 15730 9150 50  0001 C CNN
 F 3 "~" H 15800 9150 50  0001 C CNN
 	1    15800 9150
@@
 F 0 "R21" H 15870 9696 50  0000 L CNN
 F 1 "R" H 15870 9605 50  0000 L CNN
-F 2 "" V 15730 9650 50  0001 C CNN
+F 2 "Resistor_THT:R_Axial_DIN0309_L9.0mm_D3.2mm_P20.32mm_Horizontal" V 15730 9650 50  0001 C CNN
 F 3 "~" H 15800 9650 50  0001 C CNN
 	1    15800 9650
@@
 F 0 "R22" H 17220 8446 50  0000 L CNN
 F 1 "R" H 17220 8355 50  0000 L CNN
-F 2 "" V 17080 8400 50  0001 C CNN
+F 2 "Resistor_THT:R_Axial_DIN0309_L9.0mm_D3.2mm_P20.32mm_Horizontal" V 17080 8400 50  0001 C CNN
 F 3 "~" H 17150 8400 50  0001 C CNN
 	1    17150 8400
@@
 INPUT-AC
 $Comp
-L Device:R R?
+L Device:R R18
 U 1 1 5BC719BD
 P 12000 1600
-F 0 "R?" H 12070 1646 50  0000 L CNN
+F 0 "R18" H 12070 1646 50  0000 L CNN
 F 1 "R" H 12070 1555 50  0000 L CNN
 F 2 "Resistor_THT:R_Axial_DIN0309_L9.0mm_D3.2mm_P20.32mm_Horizontal" V 11930 1600 50  0001 C CNN
@@
 $EndComp
 $Comp
-L Device:R R?
+L Device:R R19
 U 1 1 5BC71C3B
 P 12000 2600
-F 0 "R?" H 12070 2646 50  0000 L CNN
+F 0 "R19" H 12070 2646 50  0000 L CNN
 F 1 "R" H 12070 2555 50  0000 L CNN
 F 2 "Resistor_THT:R_Axial_DIN0309_L9.0mm_D3.2mm_P20.32mm_Horizontal" V 11930 2600 50  0001 C CNN
@@
 $EndComp
 $Comp
-L Device:R R?
+L Device:R R23
 U 1 1 5BC729E1
 P 18900 2150
-F 0 "R?" H 18970 2196 50  0000 L CNN
+F 0 "R23" H 18970 2196 50  0000 L CNN
 F 1 "R" H 18970 2105 50  0000 L CNN
 F 2 "Resistor_THT:R_Axial_DIN0309_L9.0mm_D3.2mm_P20.32mm_Horizontal" V 18830 2150 50  0001 C CNN
@@
 	1    0    0    -1
 $EndComp
+Wire Wire Line
+	8950 7150 9550 7150
+Wire Wire Line
+	9850 7800 9850 7400
+Wire Wire Line
+	9850 7400 10250 7400
+Wire Wire Line
+	8900 7800 9850 7800
 $EndSCHEMATC

Commit message: powsupper
Parts:
- DS1: footprint LCD128*64 -> Display:AG12864E
- U1, U10, U8: footprint (none) -> Package_TO_SOT_THT:TO-220-3_Vertical
- U3: footprint (none) -> Package_DIP:DIP-8_W7.62mm_Socket_LongPads
- U4, U5, U6, U9: footprint (none) -> Package_DIP:DIP-8_W7.62mm_LongPads
Changed lines of the file:
@@
 F 0 "U1" H 4400 2092 50  0000 C CNN
 F 1 "L7805" H 4400 2001 50  0000 C CNN
-F 2 "" H 4425 1700 50  0001 L CIN
+F 2 "Package_TO_SOT_THT:TO-220-3_Vertical" H 4425 1700 50  0001 L CIN
 F 3 "http://www.st.com/content/ccc/resource/technical/document/datasheet/41/4f/b3/b0/12/d4/47/88/CD00000444.pdf/files/CD00000444.pdf/jcr:content/translations/en.CD00000444.pdf" H 4400 1800 50  0001 C CNN
 	1    4400 1850
@@
 F 0 "U3" H 7100 8200 50  0000 C CNN
 F 1 "MCP4822" H 6950 8100 50  0000 C CNN
-F 2 "" H 8050 7300 50  0001 C CNN
+F 2 "Package_DIP:DIP-8_W7.62mm_Socket_LongPads" H 8050 7300 50  0001 C CNN
 F 3 "http://ww1.microchip.com/downloads/en/DeviceDoc/20002249B.pdf" H 8050 7300 50  0001 C CNN
 	1    7250 7600
@@
 F 0 "U4" H 8991 7196 50  0000 L CNN
 F 1 "LM741" H 8991 7105 50  0000 L CNN
-F 2 "" H 8700 7200 50  0001 C CNN
+F 2 "Package_DIP:DIP-8_W7.62mm_LongPads" H 8700 7200 50  0001 C CNN
 F 3 "http://www.ti.com/lit/ds/symlink/lm741.pdf" H 8800 7300 50  0001 C CNN
 	1    8650 7150
@@
 F 0 "U5" H 9041 9396 50  0000 L CNN
 F 1 "LM741" H 9041 9305 50  0000 L CNN
-F 2 "" H 8750 9400 50  0001 C CNN
+F 2 "Package_DIP:DIP-8_W7.62mm_LongPads" H 8750 9400 50  0001 C CNN
 F 3 "http://www.ti.com/lit/ds/symlink/lm741.pdf" H 8850 9500 50  0001 C CNN
 	1    8700 9350
@@
 F 0 "U6" H 12041 8904 50  0000 L CNN
 F 1 "LM741" H 12041 8995 50  0000 L CNN
-F 2 "" H 11750 9000 50  0001 C CNN
+F 2 "Package_DIP:DIP-8_W7.62mm_LongPads" H 11750 9000 50  0001 C CNN
 F 3 "http://www.ti.com/lit/ds/symlink/lm741.pdf" H 11850 9100 50  0001 C CNN
 	1    11700 8950
@@
 F 0 "U9" H 16841 8746 50  0000 L CNN
 F 1 "LM311" H 16841 8655 50  0000 L CNN
-F 2 "" H 16500 8700 50  0001 C CNN
+F 2 "Package_DIP:DIP-8_W7.62mm_LongPads" H 16500 8700 50  0001 C CNN
 F 3 "http://www.ti.com/lit/ds/symlink/lm311.pdf" H 16500 8700 50  0001 C CNN
 	1    16500 8700
@@
 F 0 "DS1" H 3050 7650 50  0000 C CNN
 F 1 "128*64" H 3050 7550 50  0000 C CNN
-F 2 "LCD128*64" H 3300 5800 50  0001 C CIN
+F 2 "Display:AG12864E" H 3300 5800 50  0001 C CIN
 F 3 "https://www.digchip.com/datasheets/parts/datasheet/1121/AG-12864E-pdf.php" H 3500 6500 50  0001 C CNN
 	1    3300 6700
@@
 F 0 "U8" H 10400 3200 50  0000 C CNN
 F 1 "L7915" H 10400 3109 50  0000 C CNN
-F 2 "" H 10400 3150 50  0001 C CIN
+F 2 "Package_TO_SOT_THT:TO-220-3_Vertical" H 10400 3150 50  0001 C CIN
 F 3 "http://www.st.com/content/ccc/resource/technical/document/datasheet/c9/16/86/41/c7/2b/45/f2/CD00000450.pdf/files/CD00000450.pdf/jcr:content/translations/en.CD00000450.pdf" H 10400 3350 50  0001 C CNN
 	1    10400 3350
@@
 F 0 "U10" H 17300 2092 50  0000 C CNN
 F 1 "L7812" H 17300 2001 50  0000 C CNN
-F 2 "" H 17325 1700 50  0001 L CIN
+F 2 "Package_TO_SOT_THT:TO-220-3_Vertical" H 17325 1700 50  0001 L CIN
 F 3 "http://www.st.com/content/ccc/resource/technical/document/datasheet/41/4f/b3/b0/12/d4/47/88/CD00000444.pdf/files/CD00000444.pdf/jcr:content/translations/en.CD00000444.pdf" H 17300 1800 50  0001 C CNN
 	1    17300 1850
